Commit message: update(xacro): dummyプリフィックスをDummyに変更

File: cet200_description/urdf/cet200.urdf (robot description, URDF)
Before this commit: robot cet200, 32 links, 31 joints
Links:
- removed link dummy_RB_CrawlerBelt_L
- removed link dummy_RB_CrawlerBelt_R
- added link Dummy_RB_CrawlerBelt_L; visual mesh filename=package://cet200_description/meshes/crawler_belt.dae
- added link Dummy_RB_CrawlerBelt_R; visual mesh filename=package://cet200_description/meshes/crawler_belt.dae
Joints:
- removed joint dummy_LockJoint_CrawlerBelt_L
- removed joint dummy_LockJoint_CrawlerBelt_R
- removed joint dummy_LockJoint_RB_TrackFrame
- removed joint dummy_LockJoint_RB_TrackFrame_base
- removed joint dummy_LockJoint_RB_UpperStructure_RB_LidarBase
- added joint Dummy_LockJoint_CrawlerBelt_L: type fixed, parent RB_TrackFrame, child Dummy_RB_CrawlerBelt_L, origin xyz=1.6872 1.09461 0.38945 rpy=0 0 0
- added joint Dummy_LockJoint_CrawlerBelt_R: type fixed, parent RB_TrackFrame, child Dummy_RB_CrawlerBelt_R, origin xyz=1.6872 -1.09461 0.38945 rpy=0 0 0
- added joint Dummy_LockJoint_Origin: type fixed, parent TF_Origin, child RB_TrackFrame
- added joint Dummy_LockJoint_RB_TrackFrame_base: type fixed, parent RB_TrackFrame, child base_link
- added joint Dummy_LockJoint_RB_UpperStructure_RB_LidarBase: type fixed, parent RB_UpperStructure, child TF_LidarBase, origin xyz=1.17928 0.9 2.10413 rpy=0 0.7853981633974483 0, axis 0 1 0

File: cet200_description/urdf/cet200.xacro (robot description, xacro)
@@ -112,6 +112,6 @@
   <!-- Macro Crawler Belt -->
   <xacro:macro name="macro_crawler_belt" params="name:='' joint_xyz:='0 0 0'">
-    <xacro:property name="link_name" value="dummy_RB_${name}"/>
-    <joint name="dummy_LockJoint_${name}" type="fixed">
+    <xacro:property name="link_name" value="Dummy_RB_${name}"/>
+    <joint name="Dummy_LockJoint_${name}" type="fixed">
       <origin xyz="${joint_xyz}"  rpy="0 0 0" />
       <parent link="RB_TrackFrame" />
@@ -131,5 +131,5 @@
   <link name="TF_Origin" />
   <link name="base_link" />
-  <joint name="dummy_LockJoint_RB_TrackFrame" type="fixed">
+  <joint name="Dummy_LockJoint_Origin" type="fixed">
     <parent link="TF_Origin" />
     <child link="RB_TrackFrame" />
@@ -148,5 +148,5 @@
   </link>
   <!-- Handle base_link as a dummy link. ObserverFrame in AGX -->
-  <joint name="dummy_LockJoint_RB_TrackFrame_base" type="fixed">
+  <joint name="Dummy_LockJoint_RB_TrackFrame_base" type="fixed">
     <parent link="RB_TrackFrame" />
     <child link="base_link" />
@@ -239,5 +239,5 @@
   <!-- Attachments -->
   <!-- TF_LidarBase -->
-  <joint name="dummy_LockJoint_RB_UpperStructure_RB_LidarBase" type="fixed">
+  <joint name="Dummy_LockJoint_RB_UpperStructure_RB_LidarBase" type="fixed">
     <parent link="RB_UpperStructure" />
     <child link="TF_LidarBase" />
